File: pcb/garden_logger/garden_logger.sch (EAGLE design)
At the start: 0 parts

Commit message: added custom atmega328pb device to empty schematic
Parts:
- added FRAME1: FRAME-LETTER, SparkFun-Aesthetics:FRAME-LETTER
- added U$1: ATMEGA328PB_TQFP, zjembedded_eagle:ATMEGA328PB_TQFP
Other:
- note added: "Zach Jones"
