File: pcb/garden_logger/garden_logger.sch (EAGLE design)
At the start: 77 parts, among them J1 AVR_SPI_PRG_6PTH, J2 POWER_JACKPTH

Commit message: finished routing.  working on labels
Parts:
- removed ESP01: (no value), SparkFun-Connectors:M04PTH
- added J3: (no value), SparkFun-Connectors:M05PTH
- added VRAW: (no value), SparkFun-Connectors:M01PTH
Connections:
- new net N$23: J3.1, U$2.RXD
- net N$12: now also J3.3, U$2.CH_PD; no longer ESP01.3, U$2.RST
- net N$13: now also J3.2, U$2.TXD; no longer ESP01.4, U$2.RXD
- net N$6: now also J3.5, U$2.VCC; no longer ESP01.1, U$2.TXD
- net N$7: now also J3.4, U$2.RST; no longer ESP01.2, U$2.CH_PD
- net N$8: now also VRAW.1
- net VCC: no longer U$2.VCC
Changed lines of the file:
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@@
 <part name="GND8" library="supply1" deviceset="GND" device=""/>
 <part name="U$2" library="esp8266modules" deviceset="ESP01" device=""/>
-<part name="P+5" library="supply1" deviceset="VCC" device=""/>
 <part name="GND9" library="supply1" deviceset="GND" device=""/>
 <part name="I2C0" library="SparkFun-Connectors" deviceset="I2C_STANDARD" device=""/>
@@
 <part name="PROTO13" library="SparkFun-Connectors" deviceset="M08" device=""/>
 <part name="PROTO14" library="SparkFun-Connectors" deviceset="M08" device=""/>
-<part name="ESP01" library="SparkFun-Connectors" deviceset="M04" device="PTH"/>
 <part name="C10" library="SparkFun-Passives" deviceset="CAP_POL" device="PTH1" value="100uF"/>
 <part name="GND20" library="supply1" deviceset="GND" device=""/>
+<part name="VRAW" library="SparkFun-Connectors" deviceset="M01" device="PTH"/>
+<part name="J3" library="SparkFun-Connectors" deviceset="M05" device="PTH"/>
 </parts>
 <sheets>
@@
 <instance part="GND8" gate="1" x="63.5" y="127"/>
 <instance part="U$2" gate="G$1" x="289.56" y="81.28"/>
-<instance part="P+5" gate="VCC" x="314.96" y="76.2"/>
 <instance part="GND9" gate="1" x="271.78" y="99.06"/>
 <instance part="I2C0" gate="G$1" x="195.58" y="132.08"/>
@@
 <instance part="PROTO13" gate="G$1" x="299.72" y="205.74"/>
 <instance part="PROTO14" gate="G$1" x="314.96" y="205.74"/>
-<instance part="ESP01" gate="G$1" x="332.74" y="86.36" rot="R180"/>
 <instance part="C10" gate="G$1" x="-15.24" y="114.3"/>
 <instance part="GND20" gate="1" x="-15.24" y="104.14"/>
+<instance part="VRAW" gate="G$1" x="0" y="226.06" rot="R180"/>
+<instance part="J3" gate="G$1" x="322.58" y="86.36" rot="R180"/>
 </instances>
 <busses>
@@
 <pinref part="P+6" gate="VCC" pin="VCC"/>
 <wire x1="205.74" y1="116.84" x2="220.98" y2="116.84" width="0.1524" layer="91"/>
-</segment>
-<segment>
-<pinref part="U$2" gate="G$1" pin="VCC"/>
-<wire x1="304.8" y1="81.28" x2="304.8" y2="71.12" width="0.1524" layer="91"/>
-<pinref part="P+5" gate="VCC" pin="VCC"/>
-<wire x1="304.8" y1="71.12" x2="314.96" y2="71.12" width="0.1524" layer="91"/>
-<wire x1="314.96" y1="71.12" x2="314.96" y2="73.66" width="0.1524" layer="91"/>
 </segment>
 <segment>
@@
 <pinref part="F1" gate="G$1" pin="2"/>
 <wire x1="-7.62" y1="208.28" x2="-7.62" y2="210.82" width="0.1524" layer="91"/>
+<pinref part="VRAW" gate="G$1" pin="1"/>
+<wire x1="-7.62" y1="226.06" x2="-7.62" y2="210.82" width="0.1524" layer="91"/>
+<junction x="-7.62" y="210.82"/>
 </segment>
 </net>
@@
 <net name="N$6" class="0">
 <segment>
+<pinref part="U$2" gate="G$1" pin="VCC"/>
+<pinref part="J3" gate="G$1" pin="5"/>
+<wire x1="304.8" y1="81.28" x2="314.96" y2="81.28" width="0.1524" layer="91"/>
+</segment>
+</net>
+<net name="N$7" class="0">
+<segment>
+<pinref part="J3" gate="G$1" pin="4"/>
+<pinref part="U$2" gate="G$1" pin="RST"/>
+<wire x1="314.96" y1="83.82" x2="304.8" y2="83.82" width="0.1524" layer="91"/>
+</segment>
+</net>
+<net name="N$12" class="0">
+<segment>
+<pinref part="U$2" gate="G$1" pin="CH_PD"/>
+<pinref part="J3" gate="G$1" pin="3"/>
+<wire x1="304.8" y1="86.36" x2="314.96" y2="86.36" width="0.1524" layer="91"/>
+</segment>
+</net>
+<net name="N$13" class="0">
+<segment>
 <pinref part="U$2" gate="G$1" pin="TXD"/>
-<pinref part="ESP01" gate="G$1" pin="1"/>
-<wire x1="304.8" y1="88.9" x2="327.66" y2="88.9" width="0.1524" layer="91"/>
-</segment>
-</net>
-<net name="N$7" class="0">
-<segment>
-<pinref part="U$2" gate="G$1" pin="CH_PD"/>
-<pinref part="ESP01" gate="G$1" pin="2"/>
-<wire x1="304.8" y1="86.36" x2="327.66" y2="86.36" width="0.1524" layer="91"/>
-</segment>
-</net>
-<net name="N$12" class="0">
-<segment>
-<pinref part="U$2" gate="G$1" pin="RST"/>
-<pinref part="ESP01" gate="G$1" pin="3"/>
-<wire x1="304.8" y1="83.82" x2="327.66" y2="83.82" width="0.1524" layer="91"/>
-</segment>
-</net>
-<net name="N$13" class="0">
-<segment>
-<pinref part="ESP01" gate="G$1" pin="4"/>
-<wire x1="327.66" y1="81.28" x2="327.66" y2="66.04" width="0.1524" layer="91"/>
+<pinref part="J3" gate="G$1" pin="2"/>
+<wire x1="304.8" y1="88.9" x2="314.96" y2="88.9" width="0.1524" layer="91"/>
+</segment>
+</net>
+<net name="N$23" class="0">
+<segment>
+<pinref part="J3" gate="G$1" pin="1"/>
+<wire x1="314.96" y1="91.44" x2="314.96" y2="96.52" width="0.1524" layer="91"/>
+<wire x1="314.96" y1="96.52" x2="327.66" y2="96.52" width="0.1524" layer="91"/>
+<wire x1="327.66" y1="96.52" x2="327.66" y2="73.66" width="0.1524" layer="91"/>
 <pinref part="U$2" gate="G$1" pin="RXD"/>
-<wire x1="271.78" y1="81.28" x2="271.78" y2="66.04" width="0.1524" layer="91"/>
-<wire x1="271.78" y1="66.04" x2="327.66" y2="66.04" width="0.1524" layer="91"/>
-</segment>
-</net>
+<wire x1="327.66" y1="73.66" x2="271.78" y2="73.66" width="0.1524" layer="91"/>
+<wire x1="271.78" y1="73.66" x2="271.78" y2="81.28" width="0.1524" layer="91"/>
+</segment>
+</net>

Commit message: done with pcb labels
Connections:
- net N$12 renamed ESP01_CH_PD
- net N$13 renamed ESP01_TXD
- net N$23 renamed ESP01_RXD
- net N$6 renamed ESP01_VCC
- net N$7 renamed ESP01_RST
Changed lines of the file:
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@@
 </segment>
 </net>
-<net name="N$6" class="0">
+<net name="ESP01_VCC" class="0">
 <segment>
 <pinref part="U$2" gate="G$1" pin="VCC"/>
@@
 </segment>
 </net>
-<net name="N$7" class="0">
+<net name="ESP01_RST" class="0">
 <segment>
 <pinref part="J3" gate="G$1" pin="4"/>
@@
 </segment>
 </net>
-<net name="N$12" class="0">
+<net name="ESP01_CH_PD" class="0">
 <segment>
 <pinref part="U$2" gate="G$1" pin="CH_PD"/>
@@
 </segment>
 </net>
-<net name="N$13" class="0">
+<net name="ESP01_TXD" class="0">
 <segment>
 <pinref part="U$2" gate="G$1" pin="TXD"/>
@@
 </segment>
 </net>
-<net name="N$23" class="0">
+<net name="ESP01_RXD" class="0">
 <segment>
 <pinref part="J3" gate="G$1" pin="1"/>
